File: trx8020.kicad_pcb (KiCad board)
At the start: 2 copper layers, 12 parts, among them IC1 NE5534, IC2 78L10, M1 Mic

Commit message: ...
Parts:
- added C10: Capacitor, Raberix:C2, F.Cu at (76.3, 183.4)
- added C11: 100n, Raberix:C2, F.Cu at (83.4, 172.0)
- added C5: 6-22p, Raberix:C2Trim, F.Cu at (100.9, 177.7)
- added C6: 220p, Raberix:C2, F.Cu at (105.0, 178.3)
- added C7: 220p, Raberix:C2, F.Cu at (105.0, 186.3)
- added C8: 100n, Raberix:C2, F.Cu at (75.2, 174.5)
- added C9: Capacitor, Raberix:C2, F.Cu at (87.8, 183.4)
- added IC3: 78Lxx, Raberix:TO-92, F.Cu at (78.1, 172.0)
- added L1: 47u, Raberix:Inductor, F.Cu at (93.5, 185.9)
- added L2: 47u, Raberix:Inductor, F.Cu at (82.0, 185.9)
- added Q1: 6 MHz, Raberix:HC49-U, F.Cu at (100.9, 184.5)
- added R6: 100k, Raberix:R3, F.Cu at (87.9, 177.0)
- added R7: 680k, Raberix:R3, F.Cu at (108.8, 172.6)
- added R8: 100, Raberix:R3, F.Cu at (87.9, 174.5)
- added R9: 1k, Raberix:R3, F.Cu at (111.9, 180.8)
- added RP1: 10k, Raberix:RM-065, F.Cu at (108.1, 186.3)
- added T1: BC-547, Raberix:TO-92, F.Cu at (95.0, 175.1)

Commit message: ...
Parts:
- added C12: 100n, Raberix:C2, F.Cu at (38.1, 143.3)
- added C13: 1u, Raberix:C2, F.Cu at (35.6, 158.5)
- added C14: 1u, Raberix:C2, F.Cu at (35.6, 161.4)
- added IC4: SA612, Raberix:DIP-8, F.Cu at (30.5, 154.9)
- C10: value Capacitor -> 10p
- C9: value Capacitor -> 33p
- IC3: value 78Lxx -> 78L06
- moved R9 109.7 mm to (34.3, 103.3), turned to 90 degrees
- moved R7 106.1 mm to (26.0, 106.3), turned to 90 degrees
- moved RP1 104.6 mm to (39.8, 107.1), turned to 180 degrees
- moved C7 100.3 mm to (39.8, 110.1), turned to 0 degrees
- moved C6 100.1 mm to (31.8, 110.1), turned to 0 degrees
- moved Q1 94.4 mm to (37.8, 114.2), turned to 180 degrees
- moved C5 94.4 mm to (31.1, 114.2), turned to 270 degrees
- moved T1 86.2 mm to (28.6, 120.1), turned to 0 degrees
- moved L1 84.0 mm to (39.4, 121.7), turned to 270 degrees
- moved R8 76.3 mm to (27.9, 127.3), turned to 90 degrees
- moved R6 76.0 mm to (30.5, 127.3), turned to 90 degrees
- moved C9 75.7 mm to (36.8, 127.4), turned to 180 degrees
- moved C11 72.5 mm to (25.4, 128.5), turned to 90 degrees
- moved L2 67.9 mm to (39.4, 133.1), turned to 270 degrees
- moved IC3 60.8 mm to (30.5, 134.2), turned to 180 degrees
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Connections:
- IC3 pad 1: Net-(C11-Pad2) -> Net-(C8-Pad2)
- IC3 pad 3: Net-(C8-Pad2) -> Net-(C11-Pad2)
Routing:
- net Net-(C3-Pad2): track 63.2 -> 40.7 mm
- net Net-(C2-Pad2): track 15.6 -> 18.3 mm
- net Net-(C14-Pad1): track 17.3 -> 15.6 mm

Commit message: mixer II...
Parts:
- added C15: 68p, Raberix:C2, F.Cu at (70.0, 157.4)
- added C16: 68p, Raberix:C2, F.Cu at (64.1, 142.6)
- added C17: 68p, Raberix:C2, F.Cu at (59.1, 157.4)
- added C18: 68p, Raberix:C2, F.Cu at (53.2, 142.6)
- added C19: 68p, Raberix:C2, F.Cu at (46.9, 157.4)
- added C20: 100n, Raberix:C2, F.Cu at (75.8, 145.4)
- added C21: 100n, Raberix:C2, F.Cu at (73.4, 128.4)
- added C22: 1u, Raberix:C2, F.Cu at (85.2, 128.7)
- added IC5: SA612, Raberix:DIP-8, F.Cu at (79.4, 140.3)
- added IC6: 78L06, Raberix:TO-92, F.Cu at (76.7, 131.3)
- added Q2: 6MHz, Raberix:HC49-U, F.Cu at (67.4, 150.0)
- added Q3: 6MHz, Raberix:HC49-U, F.Cu at (61.6, 150.0)
- added Q4: 6MHz, Raberix:HC49-U, F.Cu at (55.8, 150.0)
- added Q5: 6MHz, Raberix:HC49-U, F.Cu at (49.9, 150.0)
Connections:
- IC4 pad 5: (no net) -> Net-(C19-Pad2)

Commit message: ...
Parts:
- added C23: 1u, Raberix:C2, F.Cu at (98.6, 85.7)
- added C24: 100n, Raberix:C1, F.Cu at (91.6, 79.9)
- added C25: 100n, Raberix:C1, F.Cu at (99.8, 94.7)
- added C26: 100n, Raberix:C1, F.Cu at (92.8, 92.1)
- added C27: 100n, Raberix:C1, F.Cu at (116.2, 85.3)
- added C28: 100n, Raberix:C1, F.Cu at (118.6, 93.7)
- added C29: 10u, Raberix:C2, F.Cu at (82.9, 83.7)
- added C30: 1u, Raberix:C2, F.Cu at (104.0, 74.8)
- added C31: 100n, Raberix:C1, F.Cu at (95.9, 111.4)
- added IC7: 78L05, Raberix:TO-92, F.Cu at (89.0, 73.8)
- added IC8: AD9850, Raberix:SSOP-28, F.Cu at (108.5, 105.5)
- added IC9: 78Lxx, Raberix:TO-92, F.Cu at (109.7, 76.6)
- added QG1: 125 MHz, Raberix:KXO-200, F.Cu at (136.9, 84.5)
- added R10: 3k9, Raberix:R3, F.Cu at (106.9, 90.4)
- added R11: 1k, Raberix:R3, F.Cu at (119.4, 101.2)
- added R12: 1k, Raberix:R3, F.Cu at (120.9, 106.3)
- added R13: 50, Raberix:R3, F.Cu at (121.1, 111.8)
- added R14: 50, Raberix:R3, F.Cu at (116.6, 117.9)
- moved C22 41.2 mm to (47.9, 111.1), turned to 270 degrees
- moved C15 35.4 mm to (47.9, 129.7), turned to 90 degrees
- moved IC5 30.7 mm to (53.1, 124.5), turned to 90 degrees
- moved IC6 29.5 mm to (53.1, 113.7), turned to 90 degrees
- moved C21 27.1 mm to (47.9, 119.4), turned to 270 degrees
- moved C20 24.9 mm to (58.2, 127.9), turned to 0 degrees
- moved Q2 20.8 mm to (55.5, 133.0), turned to 0 degrees
- moved C17 18.9 mm to (47.9, 142.1), turned to 90 degrees
- moved Q3 12.7 mm to (55.5, 138.8), turned to 180 degrees
- moved C18 11.3 mm to (63.1, 148.0), turned to 90 degrees
- moved C16 7.18 mm to (63.1, 135.5), turned to 270 degrees
- moved Q5 5.61 mm to (55.5, 150.5), turned to 180 degrees
- moved Q4 5.34 mm to (55.5, 144.7), turned to 0 degrees
- moved C19 4.40 mm to (50.5, 154.9)
- moved C2 1.27 mm to (39.0, 169.5)
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Connections:
- net Net-(C11-Pad2) renamed PWR
- IC4 pad 4: (no net) -> Net-(C19-Pad2)
- IC4 pad 5: Net-(C19-Pad2) -> (no net)
Routing:
- net PWR: track 10.4 -> 121.0 mm
- net Net-(C14-Pad1): track 15.6 -> 25.2 mm
- net Net-(C14-Pad2): track 0.00 -> 8.31 mm
- net Net-(C13-Pad2): track 0.00 -> 3.56 mm

Commit message: ...
Parts:
- added C32: 100n, Raberix:C1, F.Cu at (62.0, 113.0)
- added C33: 33p, Raberix:C1, F.Cu at (80.0, 119.6)
- added C34: 56p, Raberix:C1, F.Cu at (80.0, 129.5)
- added C35: 33p, Raberix:C1, F.Cu at (80.0, 139.2)
- added C36: 10p, Raberix:C1, F.Cu at (41.5, 110.1)
- added L3: 3.3u, Raberix:Inductor, F.Cu at (76.6, 124.7)
- added L4: 3.3u, Raberix:Inductor, F.Cu at (76.6, 134.4)
- C15, C16, C17, C18, C19, C20, C21, C22, C30, C6, C7: footprint Raberix:C2 -> Raberix:C1
- C23: value 1u -> 100n; footprint Raberix:C2 -> Raberix:C1
- C26: value 100n -> 1u
- moved IC7 84.6 mm to (95.1, 158.1), turned to 180 degrees
- moved QG1 74.4 mm to (106.9, 152.7), turned to 90 degrees
- moved C23 73.7 mm to (97.9, 159.4), turned to 90 degrees
- moved C24 68.3 mm to (98.4, 147.8), turned to 90 degrees
- moved C26 67.5 mm to (87.2, 159.4), turned to 90 degrees
- moved C27 64.8 mm to (84.2, 141.7), turned to 270 degrees
- moved C28 64.2 mm to (84.2, 147.8), turned to 270 degrees
- moved C30 61.3 mm to (109.1, 135.9), turned to 270 degrees
- moved IC9 61.2 mm to (101.2, 137.2)
- moved R13 55.6 mm to (77.2, 145.9)
- moved C29 51.7 mm to (91.7, 134.6), turned to 270 degrees
- moved C25 47.1 mm to (98.4, 141.7), turned to 90 degrees
- moved R14 46.9 mm to (77.2, 143.4)
- moved R10 44.7 mm to (94.5, 133.3), turned to 90 degrees
- moved R11 44.3 mm to (88.9, 133.3), turned to 270 degrees
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Connections:
- C23 pad 1: PWR -> Net-(C23-Pad1)
- C24 pad 1: GND -> Net-(C23-Pad1)
- C24 pad 2: Net-(C24-Pad2) -> GND
- C26 pad 1: Net-(C24-Pad2) -> PWR
- C27 pad 1: GND -> Net-(C25-Pad2)
- C27 pad 2: Net-(C25-Pad2) -> GND
- C28 pad 2: Net-(C24-Pad2) -> Net-(C23-Pad1)
- IC5 pad 6: (no net) -> Net-(C32-Pad2)
- IC7 pad 1: Net-(C24-Pad2) -> Net-(C23-Pad1)
- IC8 pad 23: Net-(C24-Pad2) -> Net-(C23-Pad1)
- IC8 pad 3: Net-(C24-Pad2) -> Net-(C23-Pad1)
- IC8 pad 4: Net-(C24-Pad2) -> Net-(C23-Pad1)
- IC8 pad 6: Net-(C24-Pad2) -> Net-(C23-Pad1)
- Q1 pad 1: GND -> Net-(C36-Pad2)
- QG1 pad 14: Net-(C24-Pad2) -> Net-(C23-Pad1)
Routing:
- net Net-(C6-Pad1): track 0.00 -> 23.6 mm
- net Net-(C5-Pad2): track 0.00 -> 20.9 mm
- net Net-(C8-Pad2): track 0.00 -> 20.5 mm
- net Net-(C19-Pad2): track 0.00 -> 13.2 mm
- net Net-(R9-Pad1): track 0.00 -> 12.5 mm
- net Net-(C18-Pad1): track 0.00 -> 10.9 mm
- net Net-(C17-Pad1): track 0.00 -> 10.9 mm
- net Net-(C16-Pad1): track 0.00 -> 10.9 mm
- net Net-(C10-Pad2): track 0.00 -> 8.15 mm
- net PWR: track 121.0 -> 128.5 mm
- net Net-(C9-Pad2): track 0.00 -> 6.35 mm
- net Net-(C15-Pad1): track 0.00 -> 6.11 mm
- net Net-(C21-Pad2): track 0.00 -> 5.97 mm
- net Net-(C19-Pad1): track 0.00 -> 5.14 mm
- net Net-(C15-Pad2): track 0.00 -> 5.09 mm
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- removed copper zone on F.Cu, net GND

Commit message: DDS
Parts:
- added C37: 27p, Raberix:C1, F.Cu at (73.5, 126.2)
- added J1: Pin_1x6, Raberix:Pin_1x6, F.Cu at (89.7, 151.1)
- added L5: 3.3u, Raberix:Inductor, F.Cu at (77.3, 121.6)
- added R15: 390, Raberix:R3, F.Cu at (77.2, 116.6)
- added R16: 390, Raberix:R3, F.Cu at (89.4, 130.4)
- added RP2: 10k, Raberix:RM-065, F.Cu at (101.6, 132.8)
- C33: value 33p -> 47p
- C34: value 56p -> 47p
- C35: value 33p -> 27p
- R13, R14: value 50 -> 100
- moved C35 21.5 mm to (97.0, 126.1), turned to 270 degrees
- moved L4 20.9 mm to (93.1, 121.6), turned to 0 degrees
- moved R13 17.7 mm to (89.4, 133.1), turned to 180 degrees
- moved C29 15.3 mm to (77.2, 129.8), turned to 0 degrees
- moved C31 13.2 mm to (101.6, 123.1)
- moved C30 13.1 mm to (106.7, 123.1)
- moved R11 10.5 mm to (78.5, 132.5), turned to 0 degrees
- moved IC9 10.3 mm to (101.6, 126.9)
- moved C34 9.77 mm to (89.2, 126.1), turned to 270 degrees
- moved L3 9.18 mm to (85.2, 121.6), turned to 0 degrees
- moved R12 7.82 mm to (78.5, 135.1), turned to 0 degrees
- moved C32 7.59 mm to (67.5, 118.2), turned to 90 degrees
- moved C33 6.60 mm to (81.3, 126.1), turned to 270 degrees
- moved QG1 6.08 mm to (101.5, 150.0)
- moved IC7 6.02 mm to (89.7, 155.6)
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Connections:
- C32 pad 1: (no net) -> Net-(C32-Pad1)
- IC8 pad 21: Net-(C35-Pad2) -> Net-(IC8-Pad21)
- IC8 pad 22: (no net) -> /RST
- IC8 pad 25: (no net) -> /DAT
- IC8 pad 7: (no net) -> /WCLK
- IC8 pad 8: (no net) -> /FQUD
- R10 pad 1: GND -> Net-(R10-Pad1)
- R13 pad 1: Net-(C35-Pad2) -> Net-(IC8-Pad21)
Routing:
- net PWR: track 128.5 -> 287.1 mm
- net Net-(C23-Pad1): track 0.00 -> 55.4 mm
- net Net-(C25-Pad2): track 0.00 -> 49.9 mm
- net /FQUD: track 0.00 -> 29.1 mm
- net /WCLK: track 0.00 -> 27.7 mm
- net /RST: track 0.00 -> 27.6 mm
- net GND: track 0.00 -> 24.2 mm
- net /DAT: track 0.00 -> 22.7 mm
- net Net-(C32-Pad1): track 0.00 -> 15.4 mm
- net Net-(C29-Pad1): track 0.00 -> 14.9 mm
- net Net-(IC8-Pad21): track 0.00 -> 14.8 mm
- net Net-(IC8-Pad20): track 0.00 -> 11.1 mm
- net Net-(C35-Pad2): track 0.00 -> 10.9 mm
- net Net-(IC8-Pad16): track 0.00 -> 9.35 mm
- net Net-(IC8-Pad9): track 0.00 -> 8.40 mm
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- added copper zone on F.Cu, net GND

Commit message: minor fix
Parts:
- moved R11 1.21 mm to (77.3, 132.5)
- moved R13 0.64 mm to (90.0, 133.1)
- moved R16 0.64 mm to (90.0, 130.4)
Routing:
- net GND: track 24.2 -> 20.2 mm
- net Net-(C29-Pad1): track 14.9 -> 14.2 mm
