File: trx8020.kicad_pcb (KiCad board)
At the start: 2 copper layers, 78 parts, among them IC1 NE5534, IC2 78L10, IC3 78L06, IC4 SA612, IC5 SA612, IC6 78L06, IC7 78L05, IC8 AD9850, IC9 78Lxx, J1 Pin_1x6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

Commit message: relays
Parts:
- added C38: 100nF, Raberix:C1, F.Cu at (73.6, 109.9)
- added C39: 22p, Raberix:C1, F.Cu at (73.6, 103.5)
- added C40: 39p, Raberix:C1, F.Cu at (83.8, 103.5)
- added C41: 39p, Raberix:C1, F.Cu at (93.9, 103.5)
- added C42: 22p, Raberix:C1, F.Cu at (104.1, 103.5)
- added L6: 56u, Raberix:Inductor, F.Cu at (78.7, 106.7)
- added L7: 68u, Raberix:Inductor, F.Cu at (88.8, 106.7)
- added L8: 56u, Raberix:Inductor, F.Cu at (99.0, 106.7)
- added REL1: AZ822-2C, Raberix:AZ822, F.Cu at (57.9, 124.3)
- added REL2: AZ822-2C, Raberix:AZ822, F.Cu at (33.3, 158.4)
- C10, C11, C12, C2, C3, C4, C8, C9: footprint Raberix:C2 -> Raberix:C1
- IC9: value 78Lxx -> 78L05
- moved C2 20.8 mm to (31.0, 188.7), turned to 90 degrees
- moved R4 18.1 mm to (36.4, 169.0), turned to 180 degrees
- moved C20 17.9 mm to (48.5, 113.9), turned to 270 degrees
- moved R5 15.3 mm to (37.6, 187.5), turned to 0 degrees
- moved C15 14.3 mm to (65.5, 131.9), turned to 0 degrees
- moved C21 11.2 mm to (51.7, 104.1)
- moved C22 9.53 mm to (50.4, 100.3)
- moved IC6 9.53 mm to (55.6, 104.1)
- moved IC5 9.36 mm to (52.9, 115.6)
- moved C13 7.73 mm to (39.4, 151.8)
- moved C12 7.31 mm to (42.0, 137.1), turned to 270 degrees
- moved IC4 7.03 mm to (34.3, 149.0)
- moved R2 6.89 mm to (27.6, 186.2), turned to 90 degrees
- moved IC1 6.83 mm to (38.5, 183.0), turned to 180 degrees
- moved C32 6.81 mm to (65.4, 111.8), turned to 270 degrees
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Connections:
- IC4 pad 1: Net-(C14-Pad2) -> Net-(IC4-Pad1)
- IC4 pad 4: Net-(C19-Pad2) -> (no net)
- IC4 pad 5: (no net) -> Net-(IC4-Pad5)
- IC5 pad 1: Net-(C15-Pad1) -> Net-(IC5-Pad1)
- IC5 pad 4: (no net) -> Net-(IC5-Pad4)
Routing:
- net Net-(C1-Pad1): track 5.59 -> 48.7 mm, vias 0 -> 1
- net Net-(C38-Pad1): track 0.00 -> 31.3 mm, vias 0 -> 1
- net Net-(IC4-Pad5): track 0.00 -> 21.0 mm
- net Net-(C3-Pad2): track 40.7 -> 21.5 mm
- net PWR: track 287.1 -> 272.8 mm
- net Net-(IC4-Pad1): track 0.00 -> 14.1 mm
- net Net-(IC5-Pad1): track 0.00 -> 14.1 mm
- net Net-(C15-Pad1): track 6.11 -> 13.5 mm
- net Net-(C41-Pad2): track 0.00 -> 6.66 mm
- net Net-(C40-Pad2): track 0.00 -> 6.66 mm
- net Net-(IC5-Pad4): track 0.00 -> 6.49 mm
- net Net-(C38-Pad2): track 0.00 -> 6.02 mm
- net Net-(C20-Pad2): track 3.43 -> 9.26 mm
- net Net-(C2-Pad2): track 18.3 -> 23.9 mm
- net Net-(C32-Pad1): track 15.4 -> 20.2 mm
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Other:
- net class Default: via_dia 0.8 -> 1; via_drill 0.4 -> 0.6

Commit message: driver
Parts:
- added C43: 100n, Raberix:C1, F.Cu at (66.3, 88.9)
- added C44: 10n, Raberix:C1, F.Cu at (66.3, 83.8)
- added IC10: 7812, Raberix:TO-220, F.Cu at (63.1, 85.1)
- added J2: DRV_OUT, Raberix:Pin_1x2, F.Cu at (69.8, 78.4)
- added R17: 1k2, Raberix:R3, F.Cu at (88.8, 90.4)
- added R18: 150, Raberix:R3, F.Cu at (88.8, 87.4)
- added R19: 10, Raberix:R3, F.Cu at (98.7, 78.6)
- added REL3: AZ822-2C, Raberix:AZ822, F.Cu at (30.2, 85.2)
- added T2: 30t:8t, Raberix:Transformer2_Amidon-T37, F.Cu at (101.3, 85.3)
- added T3: 2N2219, Raberix:TO-39, F.Cu at (88.8, 81.5)
- added T4: 1:2, Raberix:Transformer2_Amidon-T37, F.Cu at (76.2, 85.3)
Routing:
- net PWR: track 272.8 -> 340.5 mm
- net Net-(C44-Pad2): track 0.00 -> 30.0 mm
- net Net-(C43-Pad2): track 0.00 -> 29.7 mm
- net Net-(C42-Pad2): track 3.33 -> 20.5 mm
- net Net-(J2-Pad2): track 0.00 -> 11.8 mm
- net Net-(R19-Pad2): track 0.00 -> 9.82 mm
- net Net-(T3-Pad1): track 0.00 -> 7.36 mm
- net Net-(R17-Pad1): track 0.00 -> 5.94 mm
- net Net-(T2-Pad2): track 0.00 -> 3.56 mm
- net Net-(J2-Pad1): track 0.00 -> 3.11 mm
